File: PCB/PCB.kicad_sch (KiCad schematic)
At the start: 50 parts, among them IC1 SL2.1A, J1 USB_C_Receptacle_USB2.0_16P, J2 USB_C_Receptacle_USB2.0_16P, J3 USB_C_Receptacle_USB2.0_16P, J4 USB_C_Receptacle_USB2.0_16P, J5 TRRS, SW1 SW_Push, U1 PCM2902, U2 USBLC6-2SC6, U3 USBLC6-2SC6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

Commit message: fixed usb data lines + cleaned up schematic
Connections:
- net at J2.A6 (D+): now also J2.B6 (D+), U4.4 (I/O2)
- net at J2.A7 (D-): now also J2.B7 (D-), U4.6 (I/O1)
- net at J3.B6 (D+), U5.4 (I/O2): now also J3.A6 (D+)
- net at J3.B7 (D-), U5.6 (I/O1): now also J3.A7 (D-)
- net at J1.B6 (D+), U3.4 (I/O2): now also J1.A6 (D+)
- net at J1.B7 (D-), U3.6 (I/O1): now also J1.A7 (D-)
- no-connect marks 22 -> 16
Other:
- moved on the sheet: U3, U4, U5
